Commit message: Work on new automow bringup

File: automow_description/urdf/automow.urdf.xacro (robot description, xacro)
@@ -227,5 +227,5 @@
         <!-- <origin xyz="0.815 0 0.215" rpy="0 0 -0.0523598776"/> -->
         <!-- <origin xyz="0.815 0 0.215" rpy="0 0 -0.034906585"/> -->
-        <origin xyz="0.815 0 0.215" rpy="0 0 0"/>
+        <origin xyz="0.815 0 0.215" rpy="${M_PI} 0 0"/>
         <parent link="base_link" />
         <child link="laser" />

Commit message: Working on the urdf

File: automow_description/urdf/automow.urdf.xacro (robot description, xacro)
@@ -1,6 +1,4 @@
 <?xml version="1.0"?>
-<robot
-    xmlns:xacro="http://www.ros.org/wiki/xacro"
-    name="automow">
+<robot xmlns:xacro="http://www.ros.org/wiki/xacro" name="automow">
     <material name="Green">
         <color rgba="0.0 0.8 0.0 1.0"/>
@@ -33,11 +31,4 @@
      for the navigation stack to properly function -->
     <link name="base_footprint">
-        <inertial>
-        <mass value="0.0001" />
-        <origin xyz="0 0 0" />
-        <inertia ixx="0.0001" ixy="0.0" ixz="0.0"
-                 iyy="0.0001" iyz="0.0"
-                 izz="0.0001" />
-        </inertial>
         <visual>
          <origin xyz="0 0 0" rpy="0 0 0" />
@@ -225,7 +216,5 @@
     </link>
     <joint name="laser_joint" type="fixed">
-        <!-- <origin xyz="0.815 0 0.215" rpy="0 0 -0.0523598776"/> -->
-        <!-- <origin xyz="0.815 0 0.215" rpy="0 0 -0.034906585"/> -->
-        <origin xyz="0.815 0 0.215" rpy="${M_PI} 0 0"/>
+        <origin xyz="0.9 0.17 ${0.145 - clearance}" rpy="${M_PI} 0 0.785398163"/>
         <parent link="base_link" />
         <child link="laser" />
@@ -236,4 +225,7 @@
         <child link="ahrs" />
     </joint>
+    <!--
+    Kinect related links and joints
+    -->
     <link name="kinect_link">
         <xacro:default_inertial mass="0.0001"/>
@@ -252,40 +244,14 @@
         </collision>
     </link>
-    <link name="kinect_depth_frame">
-        <xacro:default_inertial mass="0.000001"/>
-    </link>
-    <link name="kinect_depth_optical_frame">
-        <xacro:default_inertial mass="0.000001"/>
-    </link>
-    <link name="kinect_rgb_frame">
-        <xacro:default_inertial mass="0.000001"/>
-    </link>
-    <link name="kinect_rgb_optical_frame">
-        <xacro:default_inertial mass="0.000001"/>
-    </link>
+    <link name="openni_camera"/>
     <joint name="base_kinect_joint" type="fixed">
-        <origin xyz="0.49  0.005 ${c_height + 0.05}" rpy="0 ${M_PI/12} 0.034906585"/>
+        <origin xyz="0.755 0 ${0.58 - clearance}" rpy="0 0 0"/>
         <parent link="base_link"/>
         <child link="kinect_link"/>
     </joint>
-    <joint name="kinect_depth_joint" type="fixed">
-        <origin xyz="0 0.018 0" rpy="0 0 0" />
-        <parent link="kinect_link" />
-        <child link="kinect_depth_frame" />
-    </joint>
-    <joint name="kinect_depth_optical_joint" type="fixed">
-        <origin xyz="0 0 0" rpy="${-M_PI/2} 0 ${-M_PI/2}"/>
-        <parent link="kinect_depth_frame" />
-        <child link="kinect_depth_optical_frame" />
-    </joint>
-    <joint name="kinect_rgb_joint" type="fixed">
-      <origin xyz="0 -0.005 0" rpy="0 0 0" />
-      <parent link="kinect_link" />
-      <child link="kinect_rgb_frame" />
-    </joint>
-    <joint name="kinect_rgb_optical_joint" type="fixed">
-      <origin xyz="0 0 0" rpy="${-M_PI/2} 0 ${-M_PI/2}"/>
-      <parent link="kinect_rgb_frame" />
-      <child link="kinect_rgb_optical_frame" />
+    <joint name="kinect_openni_joint" type="fixed">
+        <origin xyz="0 0 0" rpy="0 0 0"/>
+        <parent link="kinect_link"/>
+        <child link="openni_camera"/>
     </joint>
 </robot>

Commit message: Updated the kinect position while calibrating...

File: automow_description/urdf/automow.urdf.xacro (robot description, xacro)
@@ -251,5 +251,5 @@
     </joint>
     <joint name="kinect_openni_joint" type="fixed">
-        <origin xyz="0 0 0" rpy="0 0 0"/>
+        <origin xyz="0 0.04 0" rpy="0 0 0"/>
         <parent link="kinect_link"/>
         <child link="openni_camera"/>

Commit message: Adding the stuff for the Sick LMS1xx

File: automow_description/urdf/automow.urdf.xacro (robot description, xacro)
@@ -255,3 +255,46 @@
         <child link="openni_camera"/>
     </joint>
+    <!--
+    Bumblebee related stuff
+    -->
+    <link name="bumblebee">
+        <xacro:default_inertial mass="0.0001"/>
+ <!--        <visual>
+            <origin xyz="0 0 0" rpy="0 0 0"/>
+            <geometry>
+                <box size="0.04 0.16 0.4"/>
+            </geometry>
+        </visual>
+        <collision>
+            <origin xyz="0 0 0" rpy="0 0 0"/>
+            <geometry>
+                <box size="0.04 0.16 0.4"/>
+            </geometry>
+        </collision> -->
+    </link>
+    <joint name="bumblee_kinect_joint" type="fixed">
+        <origin xyz="0 0 0.10" rpy="0 0 0"/>
+        <parent link="kinect_link"/>
+        <child link="bumblebee"/>
+    </joint>
+<link name="sick_laser_link">
+<xacro:default_inertial mass="0.0001"/>
+        <visual>
+            <origin xyz="0 0 ${-0.15/2.0 + 0.03}" rpy="0 0 0"/>
+            <geometry>
+                <cylinder radius="${0.09/2.0}" length="0.15"/>
+            </geometry>
+        </visual>
+        <collision>
+            <origin xyz="0 0 ${-0.15/2.0 + 0.03}" rpy="0 0 0"/>
+            <geometry>
+                <cylinder radius="${0.09/2.0}" length="0.15"/>
+            </geometry>
+        </collision>
+</link>
+    <joint name="sick_laser_base_joint" type="fixed">
+        <origin xyz="0.83 -0.1525 ${0.38 - clearance}" rpy="0 0 0"/>
+        <parent link="base_link"/>
+        <child link="sick_laser_link"/>
+    </joint>
 </robot>

Commit message: Changes to the ahrs and the laser to correct inversion technique

File: automow_description/urdf/automow.urdf.xacro (robot description, xacro)
@@ -20,4 +20,5 @@
     </material>
     <xacro:property name="M_PI" value="3.14159"/>
+    <xacro:property name="to_radians" value="0.0174532925"/>
     <xacro:macro name="default_inertial" params="mass">
         <inertial>
@@ -216,10 +217,10 @@
     </link>
     <joint name="laser_joint" type="fixed">
-        <origin xyz="0.9 0.17 ${0.145 - clearance}" rpy="${M_PI} 0 0.785398163"/>
+        <origin xyz="0.9 0.17 ${0.145 - clearance}" rpy="0 0 0.785398163"/>
         <parent link="base_link" />
         <child link="laser" />
     </joint>
     <joint name="ahrs_joint" type="fixed">
-        <origin xyz="0.22 0 ${c_height - 0.02}" rpy="${M_PI} 0 0"/>
+        <origin xyz="0.22 0 ${c_height - 0.02}" rpy="0 0 0"/>
         <parent link="base_link" />
         <child link="ahrs" />
@@ -251,5 +252,5 @@
     </joint>
     <joint name="kinect_openni_joint" type="fixed">
-        <origin xyz="0 0.04 0" rpy="0 0 0"/>
+        <origin xyz="0 0.04 0" rpy="0 0 ${1.25 * to_radians}"/>
         <parent link="kinect_link"/>
         <child link="openni_camera"/>

Commit message: Committing local changes.

File: automow_description/urdf/automow.urdf.xacro (robot description, xacro)
@@ -217,10 +217,10 @@
     </link>
     <joint name="laser_joint" type="fixed">
-        <origin xyz="0.9 0.17 ${0.145 - clearance}" rpy="0 0 0.785398163"/>
+        <origin xyz="0.9 0.17 ${0.145 - clearance}" rpy="${M_PI} 0 0.785398163"/>
         <parent link="base_link" />
         <child link="laser" />
     </joint>
     <joint name="ahrs_joint" type="fixed">
-        <origin xyz="0.22 0 ${c_height - 0.02}" rpy="0 0 0"/>
+        <origin xyz="0.22 0 ${c_height - 0.02}" rpy="${M_PI} 0 0"/>
         <parent link="base_link" />
         <child link="ahrs" />

Commit message: Friday modifications for move_base

File: automow_description/urdf/automow.urdf.xacro (robot description, xacro)
@@ -222,5 +222,5 @@
     </joint>
     <joint name="ahrs_joint" type="fixed">
-        <origin xyz="0.22 0 ${c_height - 0.02}" rpy="${M_PI} 0 0"/>
+        <origin xyz="0.22 0 ${c_height - 0.02}" rpy="0 0 0"/>
         <parent link="base_link" />
         <child link="ahrs" />

Commit message: Updated URDF for new GPS and AHRS position.

File: automow_description/urdf/automow.urdf.xacro (robot description, xacro)
@@ -184,5 +184,5 @@
         <parent link="base_top"/>
         <child link="gps"/>
-        <origin xyz="0 0 0.165"/>
+        <origin xyz="0 0 0.635"/>
     </joint>
     <link name="laser">
@@ -222,6 +222,6 @@
     </joint>
     <joint name="ahrs_joint" type="fixed">
-        <origin xyz="0.22 0 ${c_height - 0.02}" rpy="0 0 0"/>
-        <parent link="base_link" />
+        <origin xyz="0.108 0 0.41275" rpy="${M_PI} 0 0"/>
+        <parent link="base_top" />
         <child link="ahrs" />
     </joint>

Commit message: Updated URDF for bumblebee frame

File: automow_description/urdf/automow.urdf.xacro (robot description, xacro)
@@ -144,5 +144,5 @@
         <parent link="base_link"/>
         <child link="deck_link"/>
-        <origin xyz="${(.73 - .215 + .06)} 0 ${d_height}"/>
+        <origin xyz="${(.73 - .215 + .06)} 0 ${d_height}" rpy="0 0 ${M_PI/4}"/>
     </joint>
     <xacro:property name="blade_diameter" value="0.356"/>
@@ -261,17 +261,13 @@
     <link name="bumblebee">
         <xacro:default_inertial mass="0.0001"/>
- <!--        <visual>
-            <origin xyz="0 0 0" rpy="0 0 0"/>
-            <geometry>
-                <box size="0.04 0.16 0.4"/>
-            </geometry>
-        </visual>
-        <collision>
-            <origin xyz="0 0 0" rpy="0 0 0"/>
-            <geometry>
-                <box size="0.04 0.16 0.4"/>
-            </geometry>
-        </collision> -->
-    </link>
+    </link>
+    <link name="bumblebee_optical">
+        <xacro:default_inertial mass="0.0001"/>
+    </link>
+    <joint name="bumblebee_optical_joint" type="fixed">
+        <origin xyz="0 0 0" rpy="${-M_PI/2} 0 ${-M_PI/2}"/>
+        <parent link="bumblebee"/>
+        <child link="bumblebee_optical"/>
+    </joint>
     <joint name="bumblee_kinect_joint" type="fixed">
         <origin xyz="0 0 0.10" rpy="0 0 0"/>

Commit message: Adding a new collada file for the lawnmower's urdf and updating the deck position

File: automow_description/urdf/automow.urdf.xacro (robot description, xacro)
@@ -17,5 +17,8 @@
     </material>
     <material name="Grey">
-        <color rgba="0.7 0.7 0.7 0.7"/>
+        <color rgba="0.7 0.7 0.7 1.0"/>
+    </material>
+    <material name="Orange">
+        <color rgba="${205/255.0} ${140/255.0} 0.0 1.0"/>
     </material>
     <xacro:property name="M_PI" value="3.14159"/>
@@ -29,21 +32,7 @@
         </inertial>
     </xacro:macro>
-    <!-- base_footprint is a ficticious frame on the ground below base_link
+    <!-- base_footprint is a fictitious frame on the ground below base_link
      for the navigation stack to properly function -->
-    <link name="base_footprint">
-        <visual>
-         <origin xyz="0 0 0" rpy="0 0 0" />
-         <geometry>
-             <box size="0.001 0.001 0.001" />
-         </geometry>
-         <material name="Green" />
-        </visual>
-        <collision>
-          <origin xyz="0 0 0" rpy="0 0 0" />
-         <geometry>
-             <box size="0.001 0.001 0.001" />
-         </geometry>
-        </collision>
-    </link>
+    <link name="base_footprint" />
     <!-- base_link is the origin for all of the coordinates on the robot.
       For our case, this will be centered under the wheels of the
@@ -60,25 +49,17 @@
         <xacro:default_inertial mass="100"/>
         <visual>
+            <origin xyz="-0.2286 0 0" rpy="0 0 0" />
+            <geometry>
+                <mesh filename="package://automow_description/meshes/lawnmower.dae"/>
+            </geometry>
+        </visual>
+        <collision>
             <origin xyz="${c1_length/2 - 0.215} 0 ${c1_height/2}" rpy="0 0 0" />
             <geometry>
                 <box size="${c1_length} ${c_width} ${c1_height}" />
             </geometry>
-            <material name="Grey" />
-        </visual>
-        <collision>
-            <origin xyz="${c1_length/2 - 0.215} 0 ${c1_height/2}" rpy="0 0 0" />
-            <geometry>
-                <box size="${c1_length} ${c_width} ${c1_height}" />
-            </geometry>
         </collision>
     </link>
     <link name="base_top">
-        <visual>
-            <origin xyz="${c2_length/2} 0 -${c2_height/2}" rpy="0 0 0" />
-            <geometry>
-                <box size="${c2_length} ${c_width} ${c2_height}" />
-            </geometry>
-            <material name="Grey" />
-        </visual>
         <collision>
             <origin xyz="${c2_length/2} 0 -${c2_height/2}" rpy="0 0 0" />
@@ -144,5 +125,5 @@
         <parent link="base_link"/>
         <child link="deck_link"/>
-        <origin xyz="${(.73 - .215 + .06)} 0 ${d_height}" rpy="0 0 ${M_PI/4}"/>
+        <origin xyz="${0.6858} 0 ${d_height}" rpy="0 0 ${-M_PI/4}"/>
     </joint>
     <xacro:property name="blade_diameter" value="0.356"/>
@@ -192,5 +173,5 @@
                 <cylinder radius="0.06" length="0.08"/>
             </geometry>
-            <material name="Red"/>
+            <material name="Orange"/>
         </visual>
         <collision>
@@ -275,23 +256,3 @@
         <child link="bumblebee"/>
     </joint>
-<link name="sick_laser_link">
-<xacro:default_inertial mass="0.0001"/>
-        <visual>
-            <origin xyz="0 0 ${-0.15/2.0 + 0.03}" rpy="0 0 0"/>
-            <geometry>
-                <cylinder radius="${0.09/2.0}" length="0.15"/>
-            </geometry>
-        </visual>
-        <collision>
-            <origin xyz="0 0 ${-0.15/2.0 + 0.03}" rpy="0 0 0"/>
-            <geometry>
-                <cylinder radius="${0.09/2.0}" length="0.15"/>
-            </geometry>
-        </collision>
-</link>
-    <joint name="sick_laser_base_joint" type="fixed">
-        <origin xyz="0.83 -0.1525 ${0.38 - clearance}" rpy="0 0 0"/>
-        <parent link="base_link"/>
-        <child link="sick_laser_link"/>
-    </joint>
 </robot>

Commit message: Updates to settings and testing of path planner

File: automow_description/urdf/automow.urdf.xacro (robot description, xacro)
@@ -198,5 +198,5 @@
     </link>
     <joint name="laser_joint" type="fixed">
-        <origin xyz="0.9 0.17 ${0.145 - clearance}" rpy="${M_PI} 0 0.785398163"/>
+        <origin xyz="0.9 0.17 ${0.3302 - clearance}" rpy="0 0 0.785398163"/>
         <parent link="base_link" />
         <child link="laser" />

Commit message: Changes from work in the field

File: automow_description/urdf/automow.urdf.xacro (robot description, xacro)
@@ -240,4 +240,5 @@
     Bumblebee related stuff
     -->
+    <link name="bumblebee_pivot"/>
     <link name="bumblebee">
         <xacro:default_inertial mass="0.0001"/>
@@ -251,8 +252,15 @@
         <child link="bumblebee_optical"/>
     </joint>
-    <joint name="bumblee_kinect_joint" type="fixed">
-        <origin xyz="0 0 0.10" rpy="0 0 0"/>
-        <parent link="kinect_link"/>
+    <joint name="bumblebee_pivot_joint" type="fixed">
+        <origin xyz="0.047625 0 0.22225" rpy="0 0 0"/>
+        <parent link="bumblebee_pivot"/>
         <child link="bumblebee"/>
     </joint>
+    <joint name="bumblebee_pivot_base_joint" type="fixed">
+        <!-- <axis xyz="0 1 0"/>
+        <limit lower="-3.14" upper="3.14159" effort="1" velocity="1"/> -->
+        <origin xyz="0.76835 0 ${0.5127625 - clearance}" rpy="0 0.57 0"/>
+        <parent link="base_link"/>
+        <child link="bumblebee_pivot"/>
+    </joint>
 </robot>
